File: Relay_Control.kicad_sch (KiCad schematic)
At the start: 8 parts, among them J13 Current Measure, Q1 BC817

Commit message: Поменял посадочное место резистора реле
Parts:
- R41: footprint Resistor_SMD:R_0805_2012Metric_Pad1.20x1.40mm_HandSolder -> Resistor_SMD:R_1210_3225Metric_Pad1.30x2.65mm_HandSolder
Changed lines of the file:
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@@
     (property "Reference" "R41" (id 0) (at 151.384 86.106 90))
     (property "Value" "60" (id 1) (at 151.384 90.17 90))
-    (property "Footprint" "Resistor_SMD:R_0805_2012Metric_Pad1.20x1.40mm_HandSolder" (id 2) (at 151.384 88.138 0)
+    (property "Footprint" "Resistor_SMD:R_1210_3225Metric_Pad1.30x2.65mm_HandSolder" (id 2) (at 151.384 88.138 0)
       (effects (font (size 1.27 1.27)) hide)
     )
